File: schematics/schematics.kicad_pcb (KiCad board)
At the start: 2 copper layers, 94 x 63.5 mm, 23 parts

Commit message: Real code for the real version of the board
Parts:
- BAT1: footprint custom:LIPOBattery Header -> custom:PowerHeader BACKSIDE
- BZ1: footprint Buzzer_Beeper:Buzzer_12x9.5RM7.6 -> Buzzer_Beeper:MagneticBuzzer_StarMicronics_QMX
- POW1: footprint custom:LIPOBattery Header -> custom:PowerHeader
- moved R3 55.3 mm to (111.0, 115.8), turned to -90 degrees
- moved TMP1 53.4 mm to (102.5, 120.0), turned to 180 degrees
- moved R1 37.7 mm to (93.0, 115.8), turned to -90 degrees
- moved R2 35.5 mm to (89.0, 126.0), turned to 90 degrees
- moved ESP32 2.91 mm to (70.8, 79.0)
- moved BAT1 2.54 mm to (110.2, 72.1), turned to -90 degrees
- moved BatteryCharger1 2.52 mm to (138.1, 67.8)
- moved BZ1 0.55 mm to (96.8, 100.0)
Connections:
- ESP32 pad 5: SDA -> RIGHT
- ESP32 pad 8: RIGHT -> SDA
Routing:
- net 3.3V: track 57.3 -> 110.6 mm, vias 0 -> 1
- net BAT: track 17.8 -> 62.8 mm, vias 0 -> 2
- net TMP: track 21.8 -> 66.3 mm
- net Net-(BAT1-+): track 93.9 -> 118.0 mm, vias 1 -> 0
- net SDA: track 43.0 -> 64.9 mm
- net RIGHT: track 70.3 -> 80.8 mm
- net LEFT: track 43.9 -> 50.6 mm
- net BUZZER: track 60.3 -> 63.8 mm
- net DOWN: track 51.4 -> 54.3 mm
- net UP: track 32.3 -> 35.2 mm
- net RXD: track 61.7 -> 64.6 mm
- net TXD: track 68.3 -> 71.2 mm
- net B: track 111.1 -> 114.0 mm
- net SCL: track 28.0 -> 26.0 mm
- net Net-(BatteryCharger1-OUT+): track 32.3 -> 30.4 mm
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